Commit message: added a sdf file

File: src/krever_controller/description/body.urdf (robot description, URDF)
Before this commit: robot Krever, 12 links, 11 joints
Links:
- link base_link: geometry collision box size=0.6 0.8 0.3; visual box size=0.8 0.6 0.3
Joints:
- removed joint base_support_joint
- removed joint tray_joint
- removed joint u1_joint
- removed joint u2_joint
- removed joint u3_joint
- added joint base_suppot_joint: type fixed, parent base_link, child support_rod, origin xyz=-0.35 0. 0.835 rpy=0.0 0.0 0.0, limit lower=0.0 upper=0.0 effort=0.0 velocity=0.0
- added joint joint_name: type fixed, parent support_rod, child tray, origin xyz=0.375 0.0 -0.465 rpy=0.0 0.0 0.0, limit lower=0.0 upper=0.0 effort=0.0 velocity=0.0
- added joint u1: type fixed, parent support_rod, child u1, origin xyz=0 0 0.555 rpy=0.0 0.0 1.57, limit lower=0.0 upper=0.0 effort=0.0 velocity=0.0
- added joint u2: type fixed, parent support_rod, child u2, origin xyz=0.25 0.35 0.555 rpy=0.0 0.0 0, limit lower=0.0 upper=0.0 effort=0.0 velocity=0.0
- added joint u3: type fixed, parent support_rod, child u3, origin xyz=0.25 -0.35 0.555 rpy=0.0 0.0 0, limit lower=0.0 upper=0.0 effort=0.0 velocity=0.0
- joint base_right_wheel_joint: origin xyz=0 -0.325 0 rpy=0 0 0 -> xyz=-0 -0.325 0 rpy=0 0 0

Commit message: added modified urdf

File: src/krever_controller/description/body.urdf (robot description, URDF)
Before this commit: robot Krever, 12 links, 11 joints
Links:
- link base_link: geometry collision box size=0.6 0.6 0.2; visual box size=0.6 0.6 0.2
- link caster_wheel1: geometry collision sphere radius=0.025; visual sphere radius=0.025
- link caster_wheel2: geometry collision sphere radius=0.025; visual sphere radius=0.025
- link left_wheel: geometry collision cylinder length=0.03 radius=0.1; visual cylinder length=0.03 radius=0.1
- link right_wheel: geometry collision cylinder length=0.03 radius=0.1; visual cylinder length=0.03 radius=0.1
- link support_rod: geometry collision box size=0.06 0.1 1.07; visual box size=0.06 0.1 1.07
- link tray: geometry collision box size=0.6 0.6 0.01; visual box size=0.6 0.6 0.01
- link u1: geometry collision box size=0.4 0.1 0.04; visual box size=0.4 0.1 0.04
Joints:
- joint base_joint: origin xyz=0 0 0.1 rpy=0 0 0 -> xyz=0 0 0.0 rpy=0 0 0
- joint base_left_wheel_joint: origin xyz=0 0.325 0 rpy=0 0 0 -> xyz=0 0.315 0.05 rpy=0 0 0
- joint base_lidar_joint: origin xyz=0 0 0.325 rpy=0 0 0 -> xyz=0 0 0.25 rpy=0 0 0
- joint base_right_wheel_joint: origin xyz=-0 -0.325 0 rpy=0 0 0 -> xyz=-0 -0.315 0.05 rpy=0 0 0
- joint base_suppot_joint: origin xyz=-0.35 0. 0.835 rpy=0.0 0.0 0.0 -> xyz=-0.265 0. 0.76 rpy=0.0 0.0 0.0
- joint body_caster_wheel_joint1: origin xyz=0.3 0 -0.05 rpy=0 0 0 -> xyz=0.25 0 0.0 rpy=0 0 0
- joint body_caster_wheel_joint2: origin xyz=-0.3 0 -0.05 rpy=0 0 0 -> xyz=-0.25 0 0.0 rpy=0 0 0
- joint joint_name: origin xyz=0.375 0.0 -0.465 rpy=0.0 0.0 0.0 -> xyz=0.27 0.0 -0.465 rpy=0.0 0.0 0.0
- joint u2: origin xyz=0.25 0.35 0.555 rpy=0.0 0.0 0 -> xyz=0.25 0.25 0.555 rpy=0.0 0.0 0
- joint u3: origin xyz=0.25 -0.35 0.555 rpy=0.0 0.0 0 -> xyz=0.25 -0.25 0.555 rpy=0.0 0.0 0
