Commit message: created sdf file and xacro description files

File: src/krever_controller/description/body.urdf.xacro (robot description, xacro)
@@ -1,5 +1,6 @@
 <?xml version="1.0"?>
-<robot name="Krever">
-<!--colors-->
+<robot name="krever" xmlns:xacro="http://www.ros.org/wiki/xacro">
+    <xacro:include filename="body_core.xacro"/>
+    <!--colors-->
     <material name="green">
         <color rgba="0 1 0 1"/>
@@ -12,27 +13,34 @@
     </material>
     <link name="base_footprint"/>
-<!--base chassis-->
+    <link name="base_footprint">
+        <inertial>
+            <mass value="1.0"/> <!-- Adjust the mass as per your robot -->
+            <inertia ixx="0.1" ixy="0.0" ixz="0.0" iyy="0.1" iyz="0.0" izz="0.1"/>
+        </inertial>
+    </link>
+    <!--base chassis-->
     <link name="base_link">
         <visual>
             <geometry>
-                <box size="0.6 0.6 0.2"/>
-            </geometry>
-            <origin xyz="0 0 0.125" rpy="0 0 0"/>
+                <box size="0.8 0.6 0.3"/>
+            </geometry>
+            <origin xyz="0 0 0.15" rpy="0 0 0"/>
             <material name="red"/>
         </visual>
         <collision>
             <geometry>
-                <box size="0.6 0.6 0.2"/>
-            </geometry>
-            <origin xyz="0 0 0.125" rpy="0 0 0"/>
+                <box size="0.8 0.6 0.3"/>
+            </geometry>
+            <origin xyz="0 0 0.15" rpy="0 0 0"/>
             <material name="red"/>
         </collision>
+        <xacro:inertial_box mass="5.0" x="0.8" y="0.6" z="0.3" origin_xyz="0 0 0.15" origin_rpy="0 0 0"/>
     </link>
     <joint name="base_joint" type="fixed">
         <parent link="base_footprint"/>
         <child link="base_link"/>
-        <origin xyz="0 0 0.0" rpy="0 0 0"/>
-    </joint>
-<!--lidar-->
+        <origin xyz="0 0 0.1" rpy="0 0 0"/>
+    </joint>
+    <!--lidar-->
     <link name="lidar">
         <visual>
@@ -50,105 +58,110 @@
             <material name="blue"/>
         </collision>
+        <xacro:inertial_cylinder mass="0.1" radius="0.1" length="0.05" origin_xyz="0 0 0" origin_rpy="0 0 0"/>
     </link>
     <joint name="base_lidar_joint" type="fixed">
         <parent link="base_link"/>
         <child link="lidar"/>
-        <origin xyz="0 0 0.25" rpy="0 0 0"/>
-    </joint>
-<!-- left wheel-->
+        <origin xyz="0 0 0.325" rpy="0 0 0"/>
+    </joint>
+    <!-- left wheel-->
     <link name="left_wheel">
         <visual>
             <geometry>
-                <cylinder radius="0.1" length="0.03"/>
-            </geometry>
-            <origin xyz="0 0 0" rpy="1.57 0 0"/>
-            <material name="green"/>
-        </visual>
-        <collision>
-            <geometry>
-                <cylinder radius="0.1" length="0.03"/>
-            </geometry>
-            <origin xyz="0 0 0" rpy="1.57 0 0"/>
-            <material name="green"/>
-        </collision>
+                <cylinder radius="0.1" length="0.05"/>
+            </geometry>
+            <origin xyz="0 0 0" rpy="1.57 0 0"/>
+            <material name="green"/>
+        </visual>
+        <collision>
+            <geometry>
+                <cylinder radius="0.1" length="0.05"/>
+            </geometry>
+            <origin xyz="0 0 0" rpy="1.57 0 0"/>
+            <material name="green"/>
+        </collision>
+        <xacro:inertial_cylinder mass="0.1" radius="0.1" length="0.05" origin_xyz="0 0 0" origin_rpy="1.57 0 0"/>
     </link>
     <joint name="base_left_wheel_joint" type="continuous">
-    <parent link="base_link"/>
+        <parent link="base_link"/>
         <child link="left_wheel"/>
-        <origin xyz="0 0.315 0.05" rpy="0 0 0"/>
+        <origin xyz="0 0.325 0" rpy="0 0 0"/>
         <axis xyz="0 1 0"/>
     </joint>
-<!--right wheel-->
+    <!--right wheel-->
     <link name="right_wheel">
         <visual>
             <geometry>
-                <cylinder radius="0.1" length="0.03"/>
-            </geometry>
-            <origin xyz="0 0 0" rpy="1.57 0 0"/>
-            <material name="green"/>
-        </visual>
-        <collision>
-            <geometry>
-                <cylinder radius="0.1" length="0.03"/>
-            </geometry>
-            <origin xyz="0 0 0" rpy="1.57 0 0"/>
-            <material name="green"/>
-        </collision>
+                <cylinder radius="0.1" length="0.05"/>
+            </geometry>
+            <origin xyz="0 0 0" rpy="1.57 0 0"/>
+            <material name="green"/>
+        </visual>
+        <collision>
+            <geometry>
+                <cylinder radius="0.1" length="0.05"/>
+            </geometry>
+            <origin xyz="0 0 0" rpy="1.57 0 0"/>
+            <material name="green"/>
+        </collision>
+        <xacro:inertial_cylinder mass="0.1" radius="0.1" length="0.05" origin_xyz="0 0 0" origin_rpy="1.57 0 0"/>
     </link>
     <joint name="base_right_wheel_joint" type="continuous">
         <parent link="base_link"/>
         <child link="right_wheel"/>
-        <origin xyz="-0 -0.315 0.05" rpy="0 0 0"/>
+        <origin xyz="0 -0.325 0" rpy="0 0 0"/>
         <axis xyz="0 1 0"/>
     </joint>
-<!-- caster wheel1 -->
+    <!-- caster wheel1 -->
     <link name="caster_wheel1">
         <visual>
             <geometry>
-                <sphere radius="0.025"/>
-            </geometry>
-            <origin xyz="0 0 0" rpy="1.57 0 0"/>
-            <material name="blue"/>
-        </visual>
-        <collision>
-            <geometry>
-                <sphere radius="0.025"/>
-            </geometry>
-            <origin xyz="0 0 0" rpy="1.57 0 0"/>
-            <material name="blue"/>
-        </collision>
+                <sphere radius="0.05"/>
+            </geometry>
+            <origin xyz="0 0 0" rpy="0 0 0"/>
+            <material name="blue"/>
+        </visual>
+        <collision>
+            <geometry>
+                <sphere radius="0.05"/>
+            </geometry>
+            <origin xyz="0 0 0" rpy="0 0 0"/>
+            <material name="blue"/>
+        </collision>
+        <xacro:inertial_sphere mass="0.08" radius="0.05" origin_xyz="0 0 0" origin_rpy="0 0 0"/>
     </link>
     <joint name="body_caster_wheel_joint1" type="fixed">
         <parent link="base_link"/>
         <child link="caster_wheel1"/>
-        <origin xyz="0.25 0 0.0" rpy="0 0 0"/>
-    </joint>
-<!-- caster wheel2 -->
+        <origin xyz="0.3 0 -0.05" rpy="0 0 0"/>
+    </joint>
+    <!-- caster wheel2 -->
     <link name="caster_wheel2">
         <visual>
             <geometry>
-                <sphere radius="0.025"/>
-            </geometry>
-            <origin xyz="0 0 0" rpy="1.57 0 0"/>
-            <material name="blue"/>
-        </visual>
-        <collision>
-            <geometry>
-                <sphere radius="0.025"/>
-            </geometry>
-            <origin xyz="0 0 0" rpy="1.57 0 0"/>
-            <material name="blue"/>
-        </collision>
+                <sphere radius="0.05"/>
+            </geometry>
+            <origin xyz="0 0 0" rpy="0 0 0"/>
+            <material name="blue"/>
+        </visual>
+        <collision>
+            <geometry>
+                <sphere radius="0.05"/>
+            </geometry>
+            <origin xyz="0 0 0" rpy="0 0 0"/>
+            <material name="blue"/>
+        </collision>
+        <xacro:inertial_sphere mass="0.08" radius="0.05" origin_xyz="0 0 0" origin_rpy="0 0 0"/>
     </link>
     <joint name="body_caster_wheel_joint2" type="fixed">
         <parent link="base_link"/>
         <child link="caster_wheel2"/>
-        <origin xyz="-0.25 0 0.0" rpy="0 0 0"/>
-    </joint>
-<!--supporint rod-->
+        <origin xyz="-0.3 0 -0.05" rpy="0 0 0"/>
+    </joint>
+    <!--supporting rod-->
     <link name="support_rod">
         <visual>
             <geometry>
-                <box size="0.06 0.1 1.07" />
+                <box size="0.1 0.1 1.07" />
             </geometry>
             <material name="LightGrey">
@@ -158,19 +171,19 @@
         <collision>
             <geometry>
-                <box size="0.06 0.1 1.07" />
-            </geometry>
-        </collision>
-    </link>
-    <joint name="base_suppot_joint" type="fixed">
-        <origin xyz="-0.265 0. 0.76" rpy="0.0 0.0 0.0"/>
+                <box size="0.1 0.1 1.07" />
+            </geometry>
+        </collision>
+        <xacro:inertial_box mass="1.0" x="0.1" y="0.1" z="1.07" origin_xyz="0 0 0" origin_rpy="0 0 0"/>
+    </link>
+    <joint name="base_support_joint" type="fixed">
+        <origin xyz="-0.35 0 0.835" rpy="0.0 0.0 0.0"/>
         <parent link="base_link"/>
         <child link="support_rod"/>
-        <limit lower="0.0" upper="0.0" effort="0.0" velocity="0.0"/>
-    </joint>
-<!--u1-->
+    </joint>
+    <!--u1-->
     <link name="u1">
         <visual>
             <geometry>
-                <box size="0.4 0.1 0.04" />
+                <box size="0.6 0.1 0.04" />
             </geometry>
             <material name="black">
@@ -180,15 +193,15 @@
         <collision>
             <geometry>
-                <box size="0.4 0.1 0.04" />
-            </geometry>
-        </collision>
-    </link>
-    <joint name="u1" type="fixed">
+                <box size="0.6 0.1 0.04" />
+            </geometry>
+        </collision>
+        <xacro:inertial_box mass="0.3" x="0.6" y="0.1" z="0.04" origin_xyz="0 0 0" origin_rpy="0 0 0"/>
+    </link>
+    <joint name="u1_joint" type="fixed">
         <origin xyz="0 0 0.555" rpy="0.0 0.0 1.57"/>
         <parent link="support_rod"/>
         <child link="u1"/>
-        <limit lower="0.0" upper="0.0" effort="0.0" velocity="0.0"/>
-    </joint>
-<!--u2-->
+    </joint>
+    <!--u2-->
     <link name="u2">
         <visual>
@@ -205,12 +218,12 @@
             </geometry>
         </collision>
-    </link>
-    <joint name="u2" type="fixed">
-        <origin xyz="0.25 0.25 0.555" rpy="0.0 0.0 0"/>
+        <xacro:inertial_box mass="0.3" x="0.6" y="0.1" z="0.04" origin_xyz="0 0 0" origin_rpy="0 0 0"/>
+    </link>
+    <joint name="u2_joint" type="fixed">
+        <origin xyz="0.25 0.35 0.555" rpy="0.0 0.0 0"/>
         <parent link="support_rod"/>
         <child link="u2"/>
-        <limit lower="0.0" upper="0.0" effort="0.0" velocity="0.0"/>
-    </joint>
-<!--u3-->
+    </joint>
+    <!--u3-->
     <link name="u3">
         <visual>
@@ -227,17 +240,17 @@
             </geometry>
         </collision>
-    </link>
-    <joint name="u3" type="fixed">
-        <origin xyz="0.25 -0.25 0.555" rpy="0.0 0.0 0"/>
+        <xacro:inertial_box mass="0.3" x="0.6" y="0.1" z="0.04" origin_xyz="0 0 0" origin_rpy="0 0 0"/>
+    </link>
+    <joint name="u3_joint" type="fixed">
+        <origin xyz="0.25 -0.35 0.555" rpy="0.0 0.0 0"/>
         <parent link="support_rod"/>
         <child link="u3"/>
-        <limit lower="0.0" upper="0.0" effort="0.0" velocity="0.0"/>
-    </joint>
-<!--tray-->
+    </joint>
+    <!--tray-->
     <link name="tray">
         <visual>
             <origin xyz="0.0 0.0 0.0" rpy="0.0 0.0 0.0"/>
             <geometry>
-                <box size="0.6 0.6 0.01"/>
+                <box size="0.65 0.8 0.01"/>
             </geometry>
             <material name="white">
@@ -248,13 +261,13 @@
             <origin xyz="0.0 0.0 0.0" rpy="0.0 0.0 0.0"/>
             <geometry>
-                <box size="0.6 0.6 0.01"/>
-            </geometry>
-        </collision>
-    </link>
-    <joint name="joint_name" type="fixed">
-        <origin xyz="0.27 0.0 -0.465" rpy="0.0 0.0 0.0"/>
+                <box size="0.65 0.8 0.01"/>
+            </geometry>
+        </collision>
+        <xacro:inertial_box mass="0.5" x="0.65" y="0.8" z="0.01" origin_xyz="0 0 0" origin_rpy="0 0 0"/>
+    </link>
+    <joint name="tray_joint" type="fixed">
+        <origin xyz="0.375 0.0 -0.465" rpy="0.0 0.0 0.0"/>
         <parent link="support_rod"/>
         <child link="tray"/>
-        <limit lower="0.0" upper="0.0" effort="0.0" velocity="0.0"/>
     </joint>
 </robot>

File: src/krever_controller/description/demo.urdf (robot description, URDF)
Before this commit: robot Krever, 12 links, 11 joints
Links:
- removed link u1
- removed link u2
- removed link u3
- added link center_rod, mass 2; collision box size=0.4 0.1 0.04; visual box size=0.4 0.1 0.04
- added link left_rod, mass 2; collision box size=0.6 0.1 0.04; visual box size=0.6 0.1 0.04
- added link right_rod, mass 2; collision box size=0.6 0.1 0.04; visual box size=0.6 0.1 0.04
- link base_footprint: mass 1.0 -> None
- link base_link: mass None -> 15.0; geometry collision box size=0.6 0.6 0.2; visual box size=0.6 0.6 0.2
- link caster_wheel1: mass None -> 0.1; geometry collision sphere radius=0.025; visual sphere radius=0.025
- link caster_wheel2: geometry collision sphere radius=0.025; visual sphere radius=0.025
- link left_wheel: mass None -> 0.8; geometry collision cylinder length=0.03 radius=0.1; visual cylinder length=0.03 radius=0.1
- link lidar: mass None -> 0.4
- link right_wheel: mass None -> 0.8; geometry collision cylinder length=0.03 radius=0.1; visual cylinder length=0.03 radius=0.1
- link support_rod: mass None -> 7; geometry collision box size=0.06 0.1 1.0; visual box size=0.06 0.1 1.0
- link tray: mass None -> 5; geometry collision box size=0.6 0.6 0.01; visual box size=0.6 0.6 0.01
Joints:
- removed joint base_support_joint
- removed joint u1_joint
- removed joint u2_joint
- removed joint u3_joint
- added joint base_suppot_joint: type fixed, parent base_link, child support_rod, origin xyz=-0.265 0. 0.76 rpy=0.0 0.0 0.0, limit lower=0.0 upper=0.0 effort=0.0 velocity=0.0
- added joint center_rod_joint: type fixed, parent support_rod, child center_rod, origin xyz=0 0 0.555 rpy=0.0 0.0 1.57, limit lower=0.0 upper=0.0 effort=0.0 velocity=0.0
- added joint left_rod_joint: type fixed, parent support_rod, child left_rod, origin xyz=0.25 0.25 0.555 rpy=0.0 0.0 0, limit lower=0.0 upper=0.0 effort=0.0 velocity=0.0
- added joint right_rod_joint: type fixed, parent support_rod, child right_rod, origin xyz=0.25 -0.25 0.555 rpy=0.0 0.0 0, limit lower=0.0 upper=0.0 effort=0.0 velocity=0.0
- joint base_joint: origin xyz=0 0 0.1 rpy=0 0 0 -> xyz=0 0 0.0 rpy=0 0 0
- joint base_left_wheel_joint: origin xyz=0 0.325 0 rpy=0 0 0 -> xyz=0 0.315 0.05 rpy=0 0 0
- joint base_lidar_joint: origin xyz=0 0 0.325 rpy=0 0 0 -> xyz=0 0 0.25 rpy=0 0 0
- joint base_right_wheel_joint: origin xyz=0 -0.325 0 rpy=0 0 0 -> xyz=-0 -0.315 0.05 rpy=0 0 0
- joint body_caster_wheel_joint1: origin xyz=0.3 0 -0.05 rpy=0 0 0 -> xyz=0.25 0 0.0 rpy=0 0 0
- joint body_caster_wheel_joint2: origin xyz=-0.3 0 -0.05 rpy=0 0 0 -> xyz=-0.25 0 0.0 rpy=0 0 0
- joint tray_joint: limit (none) -> lower=0.0 upper=0.0 effort=0.0 velocity=0.0; origin xyz=0.375 0.0 -0.465 rpy=0.0 0.0 0.0 -> xyz=0.27 0.0 -0.465 rpy=0.0 0.0 0.0
